Commit message: finally urdf model

File: src/PI5/src/manta_bot/urdf/robotassembly.urdf (robot description, URDF)
Before this commit: robot robotassembly, 8 links, 7 joints
Links:
- removed link base_footprint
- removed link laser_frame
- removed link motor_shaft__jgb37_520__chamfer1
- removed link motor_shaft__jgb37_520__chamfer1_1
- removed link root
- removed link wheel__extrude__2_
- removed link wheel__extrude__2__1
- added link lidar_link, mass 1.2633173769153754; collision mesh filename=package://manta_bot/meshes/lidar_link.stl scale=0.001 0.001 0.001; visual mesh filename=package://manta_bot/meshes/lidar_link.stl scale=0.001 0.001 0.001
- added link motor_left_1, mass 0.1340810398508418; collision mesh filename=package://manta_bot/meshes/motor_left_1.stl scale=0.001 0.001 0.001; visual mesh filename=package://manta_bot/meshes/motor_left_1.stl scale=0.001 0.001 0.001
- added link motor_right_1, mass 0.13408104001880694; collision mesh filename=package://manta_bot/meshes/motor_right_1.stl scale=0.001 0.001 0.001; visual mesh filename=package://manta_bot/meshes/motor_right_1.stl scale=0.001 0.001 0.001
- added link wheel_left_1, mass 0.6907193572776398; collision mesh filename=package://manta_bot/meshes/wheel_left_1.stl scale=0.001 0.001 0.001; visual mesh filename=package://manta_bot/meshes/wheel_left_1.stl scale=0.001 0.001 0.001
- added link wheel_right_1, mass 0.690719357277638; collision mesh filename=package://manta_bot/meshes/wheel_right_1.stl scale=0.001 0.001 0.001; visual mesh filename=package://manta_bot/meshes/wheel_right_1.stl scale=0.001 0.001 0.001
- link base_link: mass None -> 1.7931358002694335; geometry collision mesh filename=package://manta_bot/meshes/base_link.stl scale=0.001 0.001 0.001; visual mesh filename=package://manta_bot/meshes/base_link.stl scale=0.001 0.001 0.001
Joints:
- removed joint base_footprint_to_base_link_joint
- removed joint base_link_to_root_joint
- removed joint hanging_node_to_root_joint
- removed joint hanging_node_to_root_joint_1
- removed joint revolute_1
- removed joint revolute_2
- removed joint root_to_laser_frame_joint
- added joint base_link_lidar_link_to_base_link: type fixed, parent base_link, child lidar_link, origin xyz=0.0005 -0.0255 0.0705 rpy=3.1415926535897927 -0.0 0.0
- added joint base_link_motor_left_to_base_link: type fixed, parent base_link, child motor_left_1, origin xyz=-0.096 0.0675 0.006373360000000001 rpy=6.959195283221548e-16 -1.5707963267948966 0
- added joint base_link_motor_right_to_base_link: type fixed, parent base_link, child motor_right_1, origin xyz=0.096 0.06749806000000001 0.0063960300000000005 rpy=-3.1415926535897927 -1.5707963267948966 0
- added joint motor_left_1_wheel_left_to_motor_left: type continuous, parent motor_left_1, child wheel_left_1, origin xyz=-0.006999999999999999 0.0 0.005999999999999997 rpy=0.0 -0.0 0.0, axis -0.0 6.959195283221548e-16 1.0
- added joint motor_right_1_wheel_right_to_motor_right: type continuous, parent motor_right_1, child wheel_right_1, origin xyz=-0.007000000000000007 8.881784197001253e-18 0.005999999999999997 rpy=-1.9721522630525295e-31 -0.0 0.0, axis 0.0 7.753132050511999e-16 1.0

Commit message: frames of tf + lidar rotated

File: src/PI5/src/manta_bot/urdf/robotassembly.urdf (robot description, URDF)
Before this commit: robot robotassembly_1_back, 6 links, 5 joints
Joints:
- joint base_link_lidar_link_to_base_link: origin xyz=0.0005 -0.0255 0.0705 rpy=3.1415926535897927 -0.0 0.0 -> xyz=0.0005 -0.0255 0.0705 rpy=0.0 0.0 -1.5707963267948966

Commit message: save map

File: src/PI5/src/manta_bot/urdf/robotassembly.urdf (robot description, URDF)
Before this commit: robot robotassembly_1_back, 6 links, 5 joints
Links:
- added link base_footprint
Joints:
- added joint base_footprint_to_base_link: type fixed, parent base_footprint, child base_link, origin xyz=0 0 0 rpy=0 0 3.141592653589793
- joint base_link_lidar_link_to_base_link: origin xyz=0.0005 -0.0255 0.0705 rpy=0.0 0.0 -1.5707963267948966 -> xyz=0.0005 -0.0255 0.0705 rpy=3.1415926535897927 -0.0 1.5707963267948966

Commit message: implement diff drive controler

File: src/PI5/src/manta_bot/urdf/robotassembly.urdf (robot description, URDF)
Before this commit: robot robotassembly, 8 links, 7 joints
Joints:
- removed joint revolute_1
- removed joint revolute_2
- added joint left_wheel_joint: type continuous, parent motor_shaft__jgb37_520__chamfer1_1, child wheel__extrude__2__1, origin xyz=-3.46945e-18 -1.38778e-17 0.0105 rpy=1.5708 -0 -1.5708, axis 0 -1 0
- added joint right_wheel_joint: type continuous, parent motor_shaft__jgb37_520__chamfer1, child wheel__extrude__2_, origin xyz=-3.46945e-18 1.38778e-17 0.0105 rpy=1.5708 -0 -1.5708, axis 0 1 0

File: src/PI5/src/robotassembly/urdf/robotassembly.urdf (robot description, URDF)
Before this commit: robot robotassembly, 8 links, 7 joints
Joints:
- removed joint revolute_1
- removed joint revolute_2
- added joint left_wheel_joint: type continuous, parent motor_shaft__jgb37_520__chamfer1_1, child wheel__extrude__2__1, origin xyz=-3.46945e-18 -1.38778e-17 0.0105 rpy=1.5708 -0 -1.5708, axis 0 -1 0
- added joint right_wheel_joint: type continuous, parent motor_shaft__jgb37_520__chamfer1, child wheel__extrude__2_, origin xyz=-3.46945e-18 1.38778e-17 0.0105 rpy=1.5708 -0 -1.5708, axis 0 1 0

Commit message: small changes

File: src/PI5/src/manta_bot/urdf/robotassembly.urdf (robot description, URDF)
Before this commit: robot robotassembly_1_back, 7 links, 6 joints
Links:
- added link laser_frame
Joints:
- added joint laser_frame_joint: type fixed, parent lidar_link, child laser_frame, origin xyz=0 0 0 rpy=3.1415926535897927 0 -1.5707963267948966
- joint base_link_lidar_link_to_base_link: origin xyz=0.0005 -0.0255 0.0705 rpy=3.1415926535897927 -0.0 1.5707963267948966 -> xyz=0.0005 -0.0255 0.0705 rpy=3.1415926535897927 -0.0 0

Commit message: wadawd

File: src/PI5/src/manta_bot/urdf/robotassembly.urdf (robot description, URDF)
Before this commit: robot robotassembly_1_back, 8 links, 7 joints
Joints:
- joint laser_frame_joint: origin xyz=0 0 0 rpy=3.1415926535897927 0 -1.5707963267948966 -> xyz=0 0 0 rpy=3.1415926535897927 0 0

Commit message: fixed

File: src/PI5/src/manta_bot/urdf/robotassembly.urdf (robot description, URDF)
Before this commit: robot robotassembly_1_back, 8 links, 7 joints
Joints:
- joint base_footprint_to_base_link: origin xyz=0 0 0 rpy=0 0 3.141592653589793 -> xyz=0 0 0 rpy=0 0 -1.5707963267948966
- joint laser_frame_joint: origin xyz=0 0 0 rpy=3.1415926535897927 0 0 -> xyz=0 0 0 rpy=3.1415926535897927 0 -1.5707963267948966
